File: board/BasicLEDBadge.brd (EAGLE design)
At the start: 6 parts

Commit message: new board design
Parts:
- added U$1: (no value), logos:KINGCON_OUTLINE_48MM
- added U$2: (no value), logos:KINGCON_LOGO_M
- added U$3: (no value), logos:MAKERSPACE_LOGO_FULL_S
- moved U$4 51.2 mm to (7.62, 5.08), turned to 180 degrees
- moved R1 30.2 mm to (17.8, 26.7), flipped to the bottom, turned to 0 degrees
- moved JP1 30.0 mm to (17.8, 26.7), turned to 0 degrees
- moved U$5 28.7 mm to (29.2, 16.5), turned to 90 degrees
- moved LED2 24.3 mm to (26.7, 33.0), turned to 180 degrees
- moved LED1 21.6 mm to (19.1, 33.0)
Connections:
- net SW_BATT: now also U$4.3; no longer U$4.2
- net VBATT: now also U$4.2; no longer U$4.3
Routing:
- net VBATT: track 0.00 -> 50.2 mm
- net SW_BATT: track 0.00 -> 27.4 mm
- net VLED: track 0.00 -> 20.7 mm
- added copper zone on layer 16, net GND
Other:
- board outline added: 43.2 x 36.7 mm
Changed lines of the file:
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@@
 <?xml version="1.0" encoding="utf-8"?>
 <!DOCTYPE eagle SYSTEM "eagle.dtd">
-<eagle version="7.6.0">
+<eagle version="7.5.0">
 <drawing>
 <settings>
@@
 <board>
 <plain>
+<polygon width="0.4064" layer="21">
+<vertex x="5.08" y="24.13"/>
+<vertex x="15.24" y="24.13"/>
+<vertex x="37.465" y="24.13"/>
+<vertex x="40.64" y="24.13"/>
+<vertex x="40.64" y="8.89"/>
+<vertex x="5.08" y="8.89"/>
+</polygon>
+<circle x="40.64" y="5.08" radius="1.905" width="0.4064" layer="20"/>
 </plain>
 <attributes>
@@
 </autorouter>
 <elements>
-<element name="U$4" library="switch" package="JS202011CQN" value="JS202011CQN" x="54.61" y="25.4" smashed="yes"/>
-<element name="R1" library="adafruit" package="0207/9" value="" x="47.625" y="22.225" smashed="yes" rot="R90">
-<attribute name="VALUE" x="48.26" y="19.9644" size="1.27" layer="27" ratio="10" rot="R90"/>
+<element name="U$4" library="switch" package="JS202011CQN" value="JS202011CQN" x="7.62" y="5.08" smashed="yes" rot="R180"/>
+<element name="R1" library="adafruit" package="0207/9" value="" x="17.78" y="26.67" smashed="yes" rot="MR0">
+<attribute name="VALUE" x="20.0406" y="26.035" size="1.27" layer="28" ratio="10" rot="MR0"/>
 </element>
-<element name="JP1" library="SparkFun-Passives" package="PAD-JUMPER-2-NO_NO_SILK" value="JUMPER-PAD-2-NO" x="47.625" y="23.495" smashed="yes" rot="MR90"/>
-<element name="U$5" library="battery" package="KEYSTONE_3003" value="KEYSTONE_3003" x="57.15" y="10.16" smashed="yes" rot="MR180"/>
-<element name="LED1" library="adafruit" package="LED5MM" value="" x="5.08" y="16.51"/>
-<element name="LED2" library="adafruit" package="LED5MM" value="" x="24.13" y="8.89"/>
+<element name="JP1" library="SparkFun-Passives" package="PAD-JUMPER-2-NO_NO_SILK" value="JUMPER-PAD-2-NO" x="17.78" y="26.67" smashed="yes" rot="MR0"/>
+<element name="U$5" library="battery" package="KEYSTONE_3003" value="KEYSTONE_3003" x="29.21" y="16.51" smashed="yes" rot="MR90"/>
+<element name="LED1" library="adafruit" package="LED5MM" value="" x="19.05" y="33.02" smashed="yes">
+<attribute name="VALUE" x="22.2504" y="31.2166" size="1.27" layer="27" ratio="10"/>
+</element>
+<element name="LED2" library="adafruit" package="LED5MM" value="" x="26.67" y="33.02" smashed="yes" rot="R180">
+<attribute name="VALUE" x="23.4696" y="34.8234" size="1.27" layer="27" ratio="10" rot="R180"/>
+</element>
+<element name="U$1" library="logos" package="KINGCON_OUTLINE_48MM" value="" x="1.27" y="1.27"/>
+<element name="U$2" library="logos" package="KINGCON_LOGO_M" value="" x="19.05" y="7.62" rot="MR0"/>
+<element name="U$3" library="logos" package="MAKERSPACE_LOGO_FULL_S" value="" x="17.78" y="19.05" rot="MR0"/>
 </elements>
 <signals>
@@
 <contactref element="R1" pad="1"/>
 <contactref element="JP1" pad="1"/>
-<wire x1="47.625" y1="17.653" x2="47.625" y2="23.045" width="0" layer="19" extent="16-16"/>
-<wire x1="3.81" y1="16.51" x2="47.625" y2="17.653" width="0" layer="19" extent="1-1"/>
-<wire x1="22.86" y1="8.89" x2="3.81" y2="16.51" width="0" layer="19" extent="1-1"/>
+<wire x1="18.23" y1="26.67" x2="21.59" y2="26.67" width="0.4064" layer="16"/>
+<wire x1="21.59" y1="26.67" x2="22.352" y2="26.67" width="0.4064" layer="16"/>
+<wire x1="17.78" y1="33.02" x2="17.78" y2="30.48" width="0.4064" layer="16"/>
+<wire x1="17.78" y1="30.48" x2="21.59" y2="26.67" width="0.4064" layer="16"/>
+<wire x1="27.94" y1="33.02" x2="27.94" y2="32.258" width="0.4064" layer="16"/>
+<wire x1="27.94" y1="32.258" x2="22.352" y2="26.67" width="0.4064" layer="16"/>
 </signal>
 <signal name="SW_BATT">
-<contactref element="U$4" pad="2"/>
 <contactref element="R1" pad="2"/>
 <contactref element="JP1" pad="2"/>
-<wire x1="47.625" y1="23.945" x2="54.61" y2="23.749" width="0" layer="19" extent="16-16"/>
-<wire x1="47.625" y1="26.797" x2="47.625" y2="23.945" width="0" layer="19" extent="16-16"/>
+<contactref element="U$4" pad="3"/>
+<wire x1="5.1308" y1="6.731" x2="13.208" y2="14.8082" width="0.4064" layer="16"/>
+<wire x1="13.208" y1="14.8082" x2="13.208" y2="26.67" width="0.4064" layer="16"/>
+<wire x1="17.33" y1="26.67" x2="13.208" y2="26.67" width="0.4064" layer="16"/>
 </signal>
 <signal name="VBATT">
-<contactref element="U$4" pad="3"/>
 <contactref element="U$5" pad="P$2"/>
 <contactref element="U$5" pad="P$1"/>
-<wire x1="46.5963" y1="10.16" x2="57.0992" y2="23.749" width="0" layer="19" extent="1-1"/>
-<wire x1="67.7037" y1="10.16" x2="57.0992" y2="23.749" width="0" layer="19" extent="1-1"/>
+<contactref element="U$4" pad="2"/>
+<wire x1="29.21" y1="27.0637" x2="27.9527" y2="27.0637" width="0.4064" layer="16"/>
+<wire x1="27.9527" y1="27.0637" x2="10.6045" y2="9.7155" width="0.4064" layer="16"/>
+<wire x1="10.6045" y1="9.7155" x2="7.62" y2="6.731" width="0.4064" layer="16"/>
+<wire x1="29.21" y1="5.9563" x2="25.4508" y2="9.7155" width="0.4064" layer="16"/>
+<wire x1="25.4508" y1="9.7155" x2="10.6045" y2="9.7155" width="0.4064" layer="16"/>
 </signal>
 <signal name="GND">
@@
 <contactref element="LED2" pad="K"/>
 <contactref element="U$5" pad="P$3"/>
-<wire x1="25.4" y1="8.89" x2="57.15" y2="10.16" width="0" layer="19" extent="16-16"/>
-<wire x1="6.35" y1="16.51" x2="25.4" y2="8.89" width="0" layer="19" extent="1-1"/>
+<polygon width="0.4064" layer="16">
+<vertex x="1.27" y="1.27"/>
+<vertex x="1.27" y="38.1"/>
+<vertex x="44.45" y="38.1"/>
+<vertex x="44.45" y="1.27"/>
+</polygon>
 </signal>
 </signals>

Commit message: fix small issues
Parts:
- moved U$2 1.27 mm to (17.8, 7.62)
- moved U$3 1.27 mm to (16.5, 19.1)
Changed lines of the file:
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@@
 <?xml version="1.0" encoding="utf-8"?>
 <!DOCTYPE eagle SYSTEM "eagle.dtd">
-<eagle version="7.5.0">
+<eagle version="7.6.0">
 <drawing>
 <settings>
@@
 <layer number="19" name="Unrouted" color="6" fill="1" visible="yes" active="yes"/>
 <layer number="20" name="Dimension" color="15" fill="1" visible="yes" active="yes"/>
-<layer number="21" name="tPlace" color="7" fill="1" visible="yes" active="yes"/>
+<layer number="21" name="tPlace" color="7" fill="1" visible="no" active="yes"/>
 <layer number="22" name="bPlace" color="7" fill="1" visible="yes" active="yes"/>
 <layer number="23" name="tOrigins" color="15" fill="1" visible="yes" active="yes"/>
@@
 </element>
 <element name="JP1" library="SparkFun-Passives" package="PAD-JUMPER-2-NO_NO_SILK" value="JUMPER-PAD-2-NO" x="17.78" y="26.67" smashed="yes" rot="MR0"/>
-<element name="U$5" library="battery" package="KEYSTONE_3003" value="KEYSTONE_3003" x="29.21" y="16.51" smashed="yes" rot="MR90"/>
 <element name="LED1" library="adafruit" package="LED5MM" value="" x="19.05" y="33.02" smashed="yes">
 <attribute name="VALUE" x="22.2504" y="31.2166" size="1.27" layer="27" ratio="10"/>
@@
 </element>
 <element name="U$1" library="logos" package="KINGCON_OUTLINE_48MM" value="" x="1.27" y="1.27"/>
-<element name="U$2" library="logos" package="KINGCON_LOGO_M" value="" x="19.05" y="7.62" rot="MR0"/>
-<element name="U$3" library="logos" package="MAKERSPACE_LOGO_FULL_S" value="" x="17.78" y="19.05" rot="MR0"/>
+<element name="U$2" library="logos" package="KINGCON_LOGO_M" value="" x="17.78" y="7.62" rot="MR0"/>
+<element name="U$3" library="logos" package="MAKERSPACE_LOGO_FULL_S" value="" x="16.51" y="19.05" rot="MR0"/>
+<element name="U$5" library="battery" package="KEYSTONE_3003" value="KEYSTONE_3003" x="29.21" y="16.51" smashed="yes" rot="MR90"/>
 </elements>
 <signals>
@@
 </signal>
 <signal name="VBATT">
-<contactref element="U$5" pad="P$2"/>
-<contactref element="U$5" pad="P$1"/>
 <contactref element="U$4" pad="2"/>
-<wire x1="29.21" y1="27.0637" x2="27.9527" y2="27.0637" width="0.4064" layer="16"/>
 <wire x1="27.9527" y1="27.0637" x2="10.6045" y2="9.7155" width="0.4064" layer="16"/>
 <wire x1="10.6045" y1="9.7155" x2="7.62" y2="6.731" width="0.4064" layer="16"/>
+<wire x1="25.4508" y1="9.7155" x2="10.6045" y2="9.7155" width="0.4064" layer="16"/>
+<contactref element="U$5" pad="P$1"/>
+<contactref element="U$5" pad="P$2"/>
 <wire x1="29.21" y1="5.9563" x2="25.4508" y2="9.7155" width="0.4064" layer="16"/>
-<wire x1="25.4508" y1="9.7155" x2="10.6045" y2="9.7155" width="0.4064" layer="16"/>
+<wire x1="27.9527" y1="27.0637" x2="29.21" y2="27.0637" width="0.4064" layer="16"/>
 </signal>
 <signal name="GND">
 <contactref element="LED1" pad="K"/>
 <contactref element="LED2" pad="K"/>
-<contactref element="U$5" pad="P$3"/>
 <polygon width="0.4064" layer="16">
 <vertex x="1.27" y="1.27"/>
@@
 <vertex x="44.45" y="1.27"/>
 </polygon>
+<contactref element="U$5" pad="P$3"/>
 </signal>
 </signals>
