File: board/BasicLEDBadge.sch (EAGLE design)
At the start: 6 parts

Commit message: new board design
Connections:
- net SW_BATT: now also U$4.3; no longer U$4.2
- net VBATT: now also U$4.2; no longer U$4.3
Other:
- moved on the sheet: U$4
Changed lines of the file:
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@@
 <?xml version="1.0" encoding="utf-8"?>
 <!DOCTYPE eagle SYSTEM "eagle.dtd">
-<eagle version="7.6.0">
+<eagle version="7.5.0">
 <drawing>
 <settings>
@@
 </plain>
 <instances>
-<instance part="U$4" gate="G$1" x="20.32" y="43.18"/>
+<instance part="U$4" gate="G$1" x="0" y="40.64" rot="R180"/>
 <instance part="R1" gate="G$1" x="45.72" y="38.1" rot="R90"/>
 <instance part="JP1" gate="G$1" x="55.88" y="38.1" rot="R90"/>
@@
 <net name="SW_BATT" class="0">
 <segment>
-<pinref part="U$4" gate="G$1" pin="2"/>
-<wire x1="10.16" y1="43.18" x2="15.24" y2="43.18" width="0.1524" layer="91"/>
 <wire x1="10.16" y1="43.18" x2="10.16" y2="50.8" width="0.1524" layer="91"/>
 <pinref part="R1" gate="G$1" pin="2"/>
@@
 <wire x1="10.16" y1="50.8" x2="50.8" y2="50.8" width="0.1524" layer="91"/>
 <wire x1="50.8" y1="50.8" x2="50.8" y2="45.72" width="0.1524" layer="91"/>
+<pinref part="U$4" gate="G$1" pin="3"/>
+<wire x1="5.08" y1="43.18" x2="10.16" y2="43.18" width="0.1524" layer="91"/>
 </segment>
 </net>
 <net name="VBATT" class="0">
 <segment>
-<pinref part="U$4" gate="G$1" pin="3"/>
-<wire x1="10.16" y1="40.64" x2="15.24" y2="40.64" width="0.1524" layer="91"/>
 <pinref part="U$5" gate="G$1" pin="+"/>
 <wire x1="10.16" y1="40.64" x2="10.16" y2="22.86" width="0.1524" layer="91"/>
+<pinref part="U$4" gate="G$1" pin="2"/>
+<wire x1="10.16" y1="40.64" x2="5.08" y2="40.64" width="0.1524" layer="91"/>
 </segment>
 </net>
